Commit message: added maze frame creation at reset, some new attributes for the MazeEnv and some new TODO'S as well

File: data/block20.urdf (robot description, URDF)
Before this commit: robot cube.urdf, 1 links, 0 joints
Links:
- link baselink: geometry collision box size=1 20 1; visual box size=1 20 1
