Commit message: Started to prepare staff for multi target trainning

File: MazeEnv/data/goalSphere.urdf (robot description, URDF)
Before this commit: robot Sphere, 1 links, 0 joints
Links:
- link base_link: geometry collision sphere radius=0.7; visual sphere radius=0.7

Commit message: update notebooks and some other parameters in envrionment files

File: MazeEnv/data/goalSphere.urdf (robot description, URDF)
Before this commit: robot Sphere, 1 links, 0 joints
Links:
- link base_link: geometry collision sphere radius=0.7; visual sphere radius=0.6
