Commit message: Higher walls

File: MazeEnv/data/block10.urdf (robot description, URDF)
Before this commit: robot cube.urdf, 1 links, 0 joints
Links:
- link baselink: geometry collision box size=1 10 2; visual box size=1 10 2

File: MazeEnv/data/block15.urdf (robot description, URDF)
Before this commit: robot cube.urdf, 1 links, 0 joints
Links:
- link baselink: geometry collision box size=1 15 2; visual box size=1 15 2

File: MazeEnv/data/block20.urdf (robot description, URDF)
Before this commit: robot cube.urdf, 1 links, 0 joints
Links:
- link baselink: geometry collision box size=1 20 2; visual box size=1 20 2

File: MazeEnv/data/block5.urdf (robot description, URDF)
Before this commit: robot cube.urdf, 1 links, 0 joints
Links:
- link baselink: geometry collision box size=1 5 1; visual box size=1 5 2

File: MazeEnv/data/blockCube.urdf (robot description, URDF)
Before this commit: robot cube.urdf, 1 links, 0 joints
Links:
- link baselink: geometry collision box size=1 1 2; visual box size=1 1 2
